Commit message: Updated description and bringup

File: closed_loop_dalsa_description/urdf/lab_setup2.urdf.xacro (robot description, xacro)
@@ -67,5 +67,4 @@
     <plugin filename="gz_ros2_control-system" name="gz_ros2_control::GazeboSimROS2ControlPlugin">
       <parameters>$(find closed_loop_dalsa_description)/config/ros2_controllers.yaml</parameters>
-      <parameters>$(find robotiq_hande_moveit_config)/config/ros2_controllers.yaml</parameters>
     </plugin>
   </gazebo>

File: closed_loop_dalsa_description/urdf/microplate.urdf (robot description, URDF)
Before this commit: robot microplate, 1 links, 0 joints
Links:
- removed link base_link
- added link aruco, mass 0.01; collision box size=0.04 0.04 0.001; visual mesh filename=package://closed_loop_dalsa_description/meshes/aruco-42.obj scale=1 1 1
- added link microplate_link, mass 0.1; collision box size=0.127 0.085 0.015; visual mesh filename=package://closed_loop_dalsa_description/meshes/Greiner_micr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 scale=1 1 1
Joints:
- added joint microplate_to_aruco: type fixed, parent microplate_link, child aruco, origin xyz=0 0 0.015 rpy=0 0 0
