Commit message: Updated gripper to new version

File: closed_loop_dalsa_description/config/bio_lab.srdf.xacro (robot description, xacro)
@@ -7,11 +7,11 @@
     </group>
     <group name="gripper">
-        <link name="gripper_adapter" />
         <link name="gripper_body" />
-        <link name="finger1" />
-        <!-- <link name="finger2" /> -->
+        <link name="left_fingerbase" />
+        <link name="right_fingerbase" />
         <joint name="finger_joint" />
+        <joint name="finger2_joint" />
     </group>
-    <end_effector name="hand_e" parent_link="tool0" group="gripper" parent_group="ur_manipulator_tcp" />
+    <end_effector name="hand_e" parent_link="tcp_link" group="gripper" parent_group="ur_manipulator_tcp" />
     <group_state name="closed" group="gripper">
         <joint name="finger_joint" value="0.025"/>
@@ -35,14 +35,23 @@
       <joint name="finger_joint" value="0"/>
     </group_state>
-    <disable_collisions link1="wrist_3_link" link2="gripper_adapter" reason="Adjacent" />
-    <disable_collisions link1="gripper_adapter" link2="gripper_body" reason="Adjacent" />
-    <disable_collisions link1="gripper_body" link2="finger1" reason="Adjacent" />
-    <disable_collisions link1="gripper_body" link2="finger2" reason="Adjacent" />
-    <disable_collisions link1="wrist_3_link" link2="gripper_body" reason="Never" />
+    <!-- Gripper disables -->
+    <disable_collisions link1="wrist_3_link" link2="gripper_body" reason="Adjacent" />
+    <disable_collisions link1="tool0" link2="gripper_body" reason="Adjacent" />
+    <disable_collisions link1="gripper_body" link2="left_fingerbase" reason="Adjacent" />
+    <disable_collisions link1="gripper_body" link2="right_fingerbase" reason="Adjacent" />
+    <disable_collisions link1="left_fingerbase" link2="right_fingerbase" reason="Never" />
+    <disable_collisions link1="wrist_3_link" link2="left_fingerbase" reason="Never" />
+    <disable_collisions link1="wrist_3_link" link2="right_fingerbase" reason="Never" />
+    <!-- Camera disables -->
     <disable_collisions link1="gripper_body" link2="camera_mount" reason="Adjacent" />
     <disable_collisions link1="camera_mount" link2="camera_link" reason="Adjacent" />
-    <disable_collisions link1="camera_mount" link2="finger1" reason="Never" />
-    <disable_collisions link1="camera_mount" link2="finger2" reason="Never" />
+    <disable_collisions link1="camera_mount" link2="left_fingerbase" reason="Never" />
+    <disable_collisions link1="camera_mount" link2="right_fingerbase" reason="Never" />
     <disable_collisions link1="camera_link" link2="gripper_body" reason="Never" />
+    <disable_collisions link1="camera_link" link2="left_fingerbase" reason="Never" />
+    <disable_collisions link1="camera_link" link2="right_fingerbase" reason="Never" />
+    <disable_collisions link1="wrist_3_link" link2="camera_mount" reason="Never" />
+    <disable_collisions link1="wrist_3_link" link2="camera_link" reason="Never" />
+    <!-- Table & Base Disables -->
     <disable_collisions link1="base_link_inertia" link2="lab_table" reason="Adjacent"/>
     <disable_collisions link1="shoulder_link" link2="lab_table" reason="Never"/>
@@ -50,8 +59,4 @@
     <disable_collisions link1="upper_arm_link" link2="lab_table" reason="Never" />
     <disable_collisions link1="forearm_link" link2="lab_table" reason="Never" />
-    <disable_collisions link1="tool0" link2="gripper_adapter" reason="Adjacent" />
-    <disable_collisions link1="finger1" link2="finger2" reason="Never" />
-    <disable_collisions link1="gripper_adapter" link2="finger1" reason="Never" />
-    <disable_collisions link1="gripper_adapter" link2="finger2" reason="Never" />
     <disable_collisions link1="wrist_1_link" link2="lab_table" reason="Never" />
     <disable_collisions link1="wrist_2_link" link2="lab_table" reason="Never" />

File: closed_loop_dalsa_description/urdf/lab_setup.urdf.xacro (robot description, xacro)
@@ -41,5 +41,5 @@
     <origin xyz="0 0 0.751" rpy="0 0 0" />
   </xacro:ur_robot>
-  <xacro:robotiq_hande_gripper parent="tool0">
+  <xacro:robotiq_hande_gripper parent="tool0" sim_gazebo="true">
     <origin xyz="0 0 0" rpy="0 0 ${pi}"/>
   </xacro:robotiq_hande_gripper>

File: closed_loop_dalsa_description/urdf/lab_setup2.urdf.xacro (robot description, xacro)
@@ -42,5 +42,5 @@
     <origin xyz="0 0 0.75" rpy="0 0 0" />
   </xacro:ur_robot>
-  <xacro:robotiq_hande_gripper parent="tool0">
+  <xacro:robotiq_hande_gripper parent="tool0" sim_gazebo="true">
     <origin xyz="0 0 0" rpy="0 0 ${pi}"/>
   </xacro:robotiq_hande_gripper>
